File: aspen_mk1.kicad_pcb (KiCad board)
At the start: 4 copper layers, 306.4 x 103.2 mm, 150 parts, among them SW1 SW_Push, SW10 SW_Push, SW11 SW_Push, SW12 SW_Push, SW13 SW_Push, SW14 SW_Push, SW15 SW_Push, SW16 SW_Push, SW17 SW_Push, SW18 SW_Push, SW19 SW_Push, SW2 SW_Push, SW20 SW_Push, SW21 SW_Push, SW22 SW_Push, SW23 SW_Push, SW24 SW_Push, SW25 SW_Push, SW26 SW_Push, SW27 SW_Push, SW28 SW_Push, SW29 SW_Push, SW3 SW_Push, SW30 SW_Push, SW31 SW_Push, SW32 SW_Push, SW33 SW_Push, SW34 SW_Push, SW35 SW_Push, SW36 SW_Push, SW37 SW_Push, SW38 SW_Push, SW39 SW_Push, SW4 SW_Push, SW40 SW_Push, SW41 SW_Push, SW42 SW_Push, SW43 SW_Push, SW44 SW_Push, SW45 SW_Push, SW46 SW_Push, SW47 SW_Push, SW48 SW_Push, SW49 SW_Push, SW5 SW_Push, SW50 SW_Push, SW51 SW_Push, SW52 SW_Push, SW53 SW_Push, SW54 SW_Push, SW55 SW_Push, SW56 SW_Push, SW57 SW_Push, SW58 SW_Push, SW59 SW_Push, SW6 SW_Push, SW60 SW_Push, SW61 SW_Push, SW62 SW_Push, SW63 SW_Push, SW64 SW_Push, SW65 SW_Push, SW66 SW_Push, SW67 SW_Push, SW68 SW_Push, SW7 SW_Push, SW8 SW_Push, SW9 SW_Push, U1 LD1117S33TR_SOT223, U2 STM32F042C4Tx

Commit message: remove accidental proprietary model
Parts:
- removed F1: 500mA, Fuse:Fuse_1210_3225Metric
- removed USB1: Molex-0548190589, random-keyboard-parts:Molex-0548190589
- added J1: USB_C_Receptacle_USB2.0_14P, Connector_USB:USB_C_Receptacle_JAE_DX07S016JA1R1500, B.Cu at (252.3, -118.4)
- added R2: 5.1k, Resistor_SMD:R_0805_2012Metric, B.Cu at (251.5, -111.3)
- added R3: 5.1k, Resistor_SMD:R_0805_2012Metric, B.Cu at (257.4, -111.6)
- D1, D10, D11, D12, D13, D14, D15, D16, D17, D18, D19, D2, D20, D21, D22, D23, D24, D25, D26, D27, D28, D29, D3, D30, D31, D32, D33, D34, D35, D36, D37, D38, D39, D4, D40, D41, D42, D43, D44, D45, D46, D47, D48, D49, D5, D50, D51, D52, D53, D54, D55, D56, D57, D58, D59, D6, D60, D61, D62, D63, D64, D65, D66, D67, D7, D8, D9: moved to B.Cu
- moved C1 161.3 mm to (262.6, -46.5), turned to 0 degrees
- moved SW68 150.9 mm to (263.0, -54.0), turned to 90 degrees
- moved C5 89.3 mm to (257.0, -80.2), turned to 180 degrees
- moved C7 85.8 mm to (245.9, -64.3), turned to 0 degrees
- moved C8 83.9 mm to (246.7, -61.9), turned to 0 degrees
- moved C2 83.4 mm to (254.6, -77.8), turned to 180 degrees
- moved C10 78.0 mm to (247.5, -111.1), turned to 180 degrees
- moved U2 75.6 mm to (249.2, -71.4), turned to 90 degrees
- moved C6 74.9 mm to (254.8, -64.9), turned to 90 degrees
- moved R1 74.0 mm to (247.5, -108.7), turned to 180 degrees
- moved C4 68.1 mm to (242.1, -74.4)
- moved U1 66.6 mm to (250.8, -102.7), turned to -90 degrees
- moved C9 65.7 mm to (255.7, -104.4)
- moved C3 59.8 mm to (239.9, -74.4), turned to -90 degrees
- moved D61 50.9 mm to (64.5, -28.6)
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Connections:
- U2 pad 10: COL6 -> unconnected-(U2-PA0-Pad10)
- U2 pad 11: COL7 -> unconnected-(U2-PA1-Pad11)
- U2 pad 12: COL8 -> unconnected-(U2-PA2-Pad12)
- U2 pad 13: unconnected-(U2-PA3-Pad13) -> COL3
- U2 pad 14: unconnected-(U2-PA4-Pad14) -> COL2
- U2 pad 15: unconnected-(U2-PA5-Pad15) -> COL1
- U2 pad 16: unconnected-(U2-PA6-Pad16) -> COL0
- U2 pad 2: ROW0 -> ROW2
- U2 pad 25: COL9 -> COL11
- U2 pad 27: COL11 -> COL9
- U2 pad 28: COL12 -> COL8
- U2 pad 29: COL13 -> COL7
- U2 pad 30: COL14 -> COL6
- U2 pad 31: unconnected-(U2-PA10-Pad31) -> COL5
- U2 pad 32: unconnected-(U2-PA11-Pad32) -> COL4
- U2 pad 37: unconnected-(U2-PA14-Pad37) -> COL13
- U2 pad 38: unconnected-(U2-PA15-Pad38) -> COL14
- U2 pad 39: unconnected-(U2-PB3-Pad39) -> COL12
- U2 pad 4: ROW2 -> ROW0
- U2 pad 40: COL0 -> unconnected-(U2-PB4-Pad40)
- U2 pad 41: COL1 -> unconnected-(U2-PB5-Pad41)
- U2 pad 42: COL2 -> unconnected-(U2-PB6-Pad42)
- U2 pad 43: COL3 -> unconnected-(U2-PB7-Pad43)
- U2 pad 44: unconnected-(U2-PF11-Pad44) -> +3.3V
- U2 pad 45: COL4 -> unconnected-(U2-PB8-Pad45)
- U2 pad 46: COL5 -> unconnected-(U2-PB9-Pad46)
- U2 pad 5: ROW3 -> ROW4
- U2 pad 6: ROW4 -> ROW3
Routing:
- net ROW1: track 522.1 -> 361.2 mm, vias 1 -> 2
- net ROW2: track 500.5 -> 341.2 mm, vias 1 -> 2
- net ROW0: track 542.3 -> 386.4 mm, vias 1 -> 2
- net ROW3: track 478.9 -> 354.2 mm, vias 1 -> 0
- net +5V: track 148.2 -> 23.7 mm
- net +3.3V: track 40.9 -> 148.5 mm, vias 0 -> 7
- net COL1: track 229.1 -> 330.3 mm, vias 0 -> 2
- net COL6: track 118.7 -> 209.0 mm
- net D+: track 131.0 -> 45.1 mm, vias 2 -> 0
- net COL14: track 206.3 -> 120.5 mm
- net COL2: track 208.2 -> 293.4 mm
- net COL13: track 190.5 -> 105.5 mm, vias 0 -> 2
- net D-: track 130.3 -> 47.6 mm, vias 2 -> 0
- net COL7: track 97.6 -> 168.3 mm
- net COL12: track 187.5 -> 117.9 mm
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- added copper zone on B.Cu, net GND
- added copper zone on F.Cu, net GND
- removed copper zone on In1.Cu, net GND
Other:
- board size 306.4 x 103.2 mm -> 308.8 x 99.2 mm
- copper layers 4 -> 2
